File: calidus_amp/calidus/pamp.sch (KiCad schematic (older format))
At the start: 50 parts, among them U6 TDA7293, U7 TDA7293

Commit message: WIP: Updated footprints
Parts:
- removed C21: 10u, symbol Device:CP
- removed C26, C38, C39: 220u, Capacitor_THT:CP_Radial_D10.0mm_P5.00mm, symbol Device:CP
- removed R15: 20k, symbol Device:R
- removed R17, R24: 499, symbol Device:R
- added C? (x3): 10u, Capacitor_THT:CP_Radial_D5.0mm_P2.00mm, symbol Device:CP
- added C?: 220u, Capacitor_THT:CP_Radial_D6.3mm_P2.50mm, symbol Device:CP
- added R?: 20k, Resistor_THT:R_Axial_DIN0204_L3.6mm_D1.6mm_P5.08mm_Horizontal, symbol Device:R
- C20: footprint (none) -> Capacitor_THT:CP_Radial_D5.0mm_P2.00mm; Manufacturer (none) -> Multicomp:MCGPR16V106M5X11; Supplier1 (none) -> Farnell:9451056
- C27: footprint Capacitor_THT:CP_Radial_D10.0mm_P5.00mm -> Capacitor_THT:CP_Radial_D6.3mm_P2.50mm; Manufacturer Rybicon:35YXF220MEFC10X12.5 -> Rybicon:10YXF220MEFC6.3X11; Supplier1 Farnel:1144628 -> Farnel:1144609; Voltage 35V -> 10V
- R14: footprint (none) -> Resistor_THT:R_Axial_DIN0204_L3.6mm_D1.6mm_P5.08mm_Horizontal; Manufacturer (none) -> Multicomp:MF12 20K; Power 1/4 -> 1/8; Supplier1 (none) -> Farnell:9342796
Connections:
- net GNDD: now also C?.2
- net GNDS: now also C?.2
- net in_l: now also C?.2
- net in_r: now also C?.2
- net stby: now also R?.1
- net at R14.2, U6.10 (MUTE), U7.10 (MUTE): now also C?.1
- net at R16.2, U6.3 (+): now also C?.1
- net at C20.1, U6.9 (STBY), U7.9 (STBY): now also R?.2
- net at R23.2, U7.3 (+): now also C?.1
- net at R26.2: now also C?.1
Other:
- note added: "1.32 HP"
- note removed: "52m HP"
Changed lines of the file:
@@
 	2900 1800 3000 1800
 Connection ~ 2900 2400
-Wire Wire Line
-	2900 2400 2800 2400
 $Comp
 L power:GNDS #PWR015
@@
 Wire Wire Line
 	3300 1800 3400 1800
-$Comp
-L Device:R R17
-U 1 1 5C37D5D9
-P 2650 2400
-F 0 "R17" V 2261 2400 50  0000 C CNN
-F 1 "499" V 2352 2400 50  0000 C CNN
-F 2 "" V 2580 2400 50  0001 C CNN
-F 3 "~" H 2650 2400 50  0001 C CNN
-F 4 "1/4" V 2443 2400 50  0000 C CNN "Power"
-F 5 "MF" V 2534 2400 50  0000 C CNN "Type"
-	1    2650 2400
-	0    1    1    0
-$EndComp
-$Comp
-L Device:CP C26
-U 1 1 5C37D603
-P 2250 2400
-F 0 "C26" V 1905 2400 50  0000 C CNN
-F 1 "220u" V 1996 2400 50  0000 C CNN
-F 2 "Capacitor_THT:CP_Radial_D10.0mm_P5.00mm" H 2288 2250 50  0001 C CNN
-F 3 "http://www.farnell.com/datasheets/2321304.pdf" H 2250 2400 50  0001 C CNN
-F 4 "35V" V 2087 2400 50  0000 C CNN "Voltage"
-F 5 "Rybicon:35YXF220MEFC10X12.5" V 2250 2400 50  0001 C CNN "Manufacturer"
-F 6 "Farnel:1144628" V 2250 2400 50  0001 C CNN "Supplier1"
-	1    2250 2400
-	0    1    1    0
-$EndComp
-Wire Wire Line
-	2400 2400 2500 2400
 Wire Wire Line
 	1950 2400 2100 2400
@@
 1.44 SHP
 Text Notes 2100 1800 0    50   ~ 0
-52m HP
+1.32 HP
 $Comp
 L Device:CP C25
@@
 	2900 5200 3000 5200
 Connection ~ 2900 5800
-Wire Wire Line
-	2900 5800 2800 5800
 $Comp
 L power:GNDS #PWR024
@@
 	3300 5200 3400 5200
 Wire Wire Line
-	2400 5800 2500 5800
-Wire Wire Line
 	1950 5800 2100 5800
 Text HLabel 1950 5800 0    50   Input ~ 0
@@
 1.44 SHP
 Text Notes 2100 5200 0    50   ~ 0
-52m HP
+1.32 HP
 Wire Wire Line
 	4100 5550 4100 5500
@@
 F 0 "C20" H 6217 1641 50  0000 L CNN
 F 1 "10u" H 6217 1550 50  0000 L CNN
-F 2 "" H 6138 1400 50  0001 C CNN
-F 3 "~" H 6100 1550 50  0001 C CNN
+F 2 "Capacitor_THT:CP_Radial_D5.0mm_P2.00mm" H 6138 1400 50  0001 C CNN
+F 3 "http://www.farnell.com/datasheets/1723232.pdf" H 6100 1550 50  0001 C CNN
 F 4 "16V" H 6217 1459 50  0000 L CNN "Voltage"
+F 5 "Multicomp:MCGPR16V106M5X11" H 6100 1550 50  0001 C CNN "Manufacturer"
+F 6 "Farnell:9451056" H 6100 1550 50  0001 C CNN "Supplier1"
 	1    6100 1550
 	-1   0    0    -1
@@
 F 0 "R14" V 6261 1000 50  0000 C CNN
 F 1 "20k" V 6352 1000 50  0000 C CNN
-F 2 "" V 6580 1000 50  0001 C CNN
-F 3 "~" H 6650 1000 50  0001 C CNN
-F 4 "1/4" V 6443 1000 50  0000 C CNN "Power"
+F 2 "Resistor_THT:R_Axial_DIN0204_L3.6mm_D1.6mm_P5.08mm_Horizontal" V 6580 1000 50  0001 C CNN
+F 3 "http://www.farnell.com/datasheets/1716726.pdf" H 6650 1000 50  0001 C CNN
+F 4 "1/8" V 6443 1000 50  0000 C CNN "Power"
 F 5 "C" V 6534 1000 50  0000 C CNN "Type"
+F 6 "Multicomp:MF12 20K" V 6650 1000 50  0001 C CNN "Manufacturer"
+F 7 "Farnell:9342796" V 6650 1000 50  0001 C CNN "Supplier1"
 	1    6650 1000
 	0    1    1    0
@@
 $EndComp
 $Comp
-L Device:CP C21
-U 1 1 5C46A2D8
-P 6400 1550
-F 0 "C21" H 6282 1641 50  0000 R CNN
-F 1 "10u" H 6282 1550 50  0000 R CNN
-F 2 "" H 6438 1400 50  0001 C CNN
-F 3 "~" H 6400 1550 50  0001 C CNN
-F 4 "16V" H 6282 1459 50  0000 R CNN "Voltage"
-	1    6400 1550
-	-1   0    0    -1
-$EndComp
-$Comp
 L Device:R R28
 U 1 1 5C46AB3E
@@
 $EndComp
 $Comp
-L Device:R R15
-U 1 1 5C46C066
-P 7150 1300
-F 0 "R15" V 7265 1300 50  0000 C CNN
-F 1 "20k" V 7356 1300 50  0000 C CNN
-F 2 "" V 7080 1300 50  0001 C CNN
-F 3 "~" H 7150 1300 50  0001 C CNN
-F 4 "1/4" V 7447 1300 50  0000 C CNN "Power"
-F 5 "C" V 7538 1300 50  0000 C CNN "Type"
-	1    7150 1300
-	0    1    1    0
-$EndComp
-$Comp
 L Device:C C36
 U 1 1 5C47384F
@@
 $EndComp
 $Comp
-L Device:R R24
-U 1 1 5C483D2D
-P 2650 5800
-F 0 "R24" V 2261 5800 50  0000 C CNN
-F 1 "499" V 2352 5800 50  0000 C CNN
-F 2 "" V 2580 5800 50  0001 C CNN
-F 3 "~" H 2650 5800 50  0001 C CNN
-F 4 "1/4" V 2443 5800 50  0000 C CNN "Power"
-F 5 "MF" V 2534 5800 50  0000 C CNN "Type"
-	1    2650 5800
-	0    1    1    0
-$EndComp
-$Comp
 L Device:R R26
 U 1 1 5C483DC7
@@
 Wire Wire Line
 	9200 1600 9300 1600
-Wire Wire Line
-	10500 1200 10500 1150
 Wire Wire Line
 	9300 1100 9900 1100
@@
 F 0 "C27" V 2413 2600 50  0000 C CNN
 F 1 "220u" V 2504 2600 50  0000 C CNN
-F 2 "Capacitor_THT:CP_Radial_D10.0mm_P5.00mm" H 2288 2450 50  0001 C CNN
+F 2 "Capacitor_THT:CP_Radial_D6.3mm_P2.50mm" H 2288 2450 50  0001 C CNN
 F 3 "http://www.farnell.com/datasheets/2321304.pdf" H 2250 2600 50  0001 C CNN
-F 4 "35V" V 2595 2600 50  0000 C CNN "Voltage"
-F 5 "Rybicon:35YXF220MEFC10X12.5" V 2250 2600 50  0001 C CNN "Manufacturer"
-F 6 "Farnel:1144628" V 2250 2600 50  0001 C CNN "Supplier1"
+F 4 "10V" V 2595 2600 50  0000 C CNN "Voltage"
+F 5 "Rybicon:10YXF220MEFC6.3X11" V 2250 2600 50  0001 C CNN "Manufacturer"
+F 6 "Farnel:1144609" V 2250 2600 50  0001 C CNN "Supplier1"
 	1    2250 2600
-	0    1    1    0
-$EndComp
-$Comp
-L Device:CP C38
-U 1 1 5C5E631C
-P 2250 5800
-F 0 "C38" V 1905 5800 50  0000 C CNN
-F 1 "220u" V 1996 5800 50  0000 C CNN
-F 2 "Capacitor_THT:CP_Radial_D10.0mm_P5.00mm" H 2288 5650 50  0001 C CNN
-F 3 "http://www.farnell.com/datasheets/2321304.pdf" H 2250 5800 50  0001 C CNN
-F 4 "35V" V 2087 5800 50  0000 C CNN "Voltage"
-F 5 "Rybicon:35YXF220MEFC10X12.5" V 2250 5800 50  0001 C CNN "Manufacturer"
-F 6 "Farnel:1144628" V 2250 5800 50  0001 C CNN "Supplier1"
-	1    2250 5800
-	0    1    1    0
-$EndComp
-$Comp
-L Device:CP C39
-U 1 1 5C5E6449
-P 2250 6000
-F 0 "C39" V 2413 6000 50  0000 C CNN
-F 1 "220u" V 2504 6000 50  0000 C CNN
-F 2 "Capacitor_THT:CP_Radial_D10.0mm_P5.00mm" H 2288 5850 50  0001 C CNN
-F 3 "http://www.farnell.com/datasheets/2321304.pdf" H 2250 6000 50  0001 C CNN
-F 4 "35V" V 2595 6000 50  0000 C CNN "Voltage"
-F 5 "Rybicon:35YXF220MEFC10X12.5" V 2250 6000 50  0001 C CNN "Manufacturer"
-F 6 "Farnel:1144628" V 2250 6000 50  0001 C CNN "Supplier1"
-	1    2250 6000
 	0    1    1    0
 $EndComp
@@
 	-1   0    0    -1
 $EndComp
-Connection ~ 10500 1150
-Wire Wire Line
-	10500 1150 10500 1100
 $Comp
 L Device:CP C24
@@
 	-1   0    0    -1
 $EndComp
+Wire Wire Line
+	10500 1100 10500 1200
+$Comp
+L Device:CP C?
+U 1 1 5C4C9B48
+P 6400 1550
+F 0 "C?" H 6282 1641 50  0000 R CNN
+F 1 "10u" H 6282 1550 50  0000 R CNN
+F 2 "Capacitor_THT:CP_Radial_D5.0mm_P2.00mm" H 6438 1400 50  0001 C CNN
+F 3 "http://www.farnell.com/datasheets/1723232.pdf" H 6400 1550 50  0001 C CNN
+F 4 "16V" H 6282 1459 50  0000 R CNN "Voltage"
+F 5 "Multicomp:MCGPR16V106M5X11" H 6400 1550 50  0001 C CNN "Manufacturer"
+F 6 "Farnell:9451056" H 6400 1550 50  0001 C CNN "Supplier1"
+	1    6400 1550
+	-1   0    0    -1
+$EndComp
+Wire Wire Line
+	2400 2400 2900 2400
+$Comp
+L Device:CP C?
+U 1 1 5C4E1EBF
+P 2250 2400
+AR Path="/5C37BC48/5C4E1EBF" Ref="C?"  Part="1"
+AR Path="/5C4751C0/5C4E1EBF" Ref="C?"  Part="1"
+AR Path="/5C37BC7C/5C4E1EBF" Ref="C?"  Part="1"
+F 0 "C?" V 1905 2400 50  0000 C CNN
+F 1 "10u" V 1996 2400 50  0000 C CNN
+F 2 "Capacitor_THT:CP_Radial_D5.0mm_P2.00mm" H 2288 2250 50  0001 C CNN
+F 3 "http://www.farnell.com/datasheets/2124421.pdf" H 2250 2400 50  0001 C CNN
+F 4 "50V" V 2087 2400 50  0000 C CNN "Voltage"
+F 5 "Rybicon:50YXF10MEFC5X11" H 2250 2400 50  0001 C CNN "Manufacturer"
+F 6 "Farnell:1144632" H 2250 2400 50  0001 C CNN "Supplier1"
+	1    2250 2400
+	0    1    1    0
+$EndComp
+$Comp
+L Device:CP C?
+U 1 1 5C4ED50B
+P 2250 5800
+AR Path="/5C37BC48/5C4ED50B" Ref="C?"  Part="1"
+AR Path="/5C4751C0/5C4ED50B" Ref="C?"  Part="1"
+AR Path="/5C37BC7C/5C4ED50B" Ref="C?"  Part="1"
+F 0 "C?" V 1905 5800 50  0000 C CNN
+F 1 "10u" V 1996 5800 50  0000 C CNN
+F 2 "Capacitor_THT:CP_Radial_D5.0mm_P2.00mm" H 2288 5650 50  0001 C CNN
+F 3 "http://www.farnell.com/datasheets/2124421.pdf" H 2250 5800 50  0001 C CNN
+F 4 "50V" V 2087 5800 50  0000 C CNN "Voltage"
+F 5 "Rybicon:50YXF10MEFC5X11" H 2250 5800 50  0001 C CNN "Manufacturer"
+F 6 "Farnell:1144632" H 2250 5800 50  0001 C CNN "Supplier1"
+	1    2250 5800
+	0    1    1    0
+$EndComp
+Wire Wire Line
+	2400 5800 2900 5800
+$Comp
+L Device:CP C?
+U 1 1 5C4F6242
+P 2250 6000
+F 0 "C?" V 2413 6000 50  0000 C CNN
+F 1 "220u" V 2504 6000 50  0000 C CNN
+F 2 "Capacitor_THT:CP_Radial_D6.3mm_P2.50mm" H 2288 5850 50  0001 C CNN
+F 3 "http://www.farnell.com/datasheets/2321304.pdf" H 2250 6000 50  0001 C CNN
+F 4 "10V" V 2595 6000 50  0000 C CNN "Voltage"
+F 5 "Rybicon:10YXF220MEFC6.3X11" V 2250 6000 50  0001 C CNN "Manufacturer"
+F 6 "Farnel:1144609" V 2250 6000 50  0001 C CNN "Supplier1"
+	1    2250 6000
+	0    1    1    0
+$EndComp
+$Comp
+L Device:R R?
+U 1 1 5C4F9DF0
+P 7150 1300
+F 0 "R?" V 7265 1300 50  0000 C CNN
+F 1 "20k" V 7356 1300 50  0000 C CNN
+F 2 "Resistor_THT:R_Axial_DIN0204_L3.6mm_D1.6mm_P5.08mm_Horizontal" V 7080 1300 50  0001 C CNN
+F 3 "http://www.farnell.com/datasheets/1716726.pdf" H 7150 1300 50  0001 C CNN
+F 4 "1/8" V 7447 1300 50  0000 C CNN "Power"
+F 5 "C" V 7538 1300 50  0000 C CNN "Type"
+F 6 "Multicomp:MF12 20K" V 7150 1300 50  0001 C CNN "Manufacturer"
+F 7 "Farnell:9342796" V 7150 1300 50  0001 C CNN "Supplier1"
+	1    7150 1300
+	0    1    1    0
+$EndComp
 $EndSCHEMATC

Commit message: WIP: component footprint assignment.
Signed-off-by: Nenad Radulovic <nenad.b.radulovic@gmail.com>
Parts:
- added C?: 220p, Capacitor_THT:C_Disc_D3.0mm_W1.6mm_P2.50mm, symbol Device:C
- added R?: 499, Resistor_THT:R_Axial_DIN0207_L6.3mm_D2.5mm_P7.62mm_Horizontal, symbol Device:R
- C17: renamed from C31; footprint (none) -> Capacitor_THT:C_Disc_D3.0mm_W1.6mm_P2.50mm
- C18: renamed from C40; footprint (none) -> Capacitor_THT:C_Disc_D3.0mm_W1.6mm_P2.50mm
- C21: renamed from C35; footprint (none) -> Capacitor_THT:C_Rect_L7.0mm_W2.5mm_P5.00mm
- C22: renamed from C41; footprint (none) -> Capacitor_THT:C_Rect_L7.0mm_W2.5mm_P5.00mm
- C23: renamed from C36; footprint (none) -> Capacitor_THT:C_Rect_L7.0mm_W2.5mm_P5.00mm
- C24: renamed from C42; footprint (none) -> Capacitor_THT:C_Rect_L7.0mm_W2.5mm_P5.00mm
- C27: renamed from C17; footprint (none) -> Capacitor_THT:C_Rect_L7.0mm_W2.5mm_P5.00mm
- C28: renamed from C22; footprint (none) -> Capacitor_THT:C_Rect_L7.0mm_W2.5mm_P5.00mm
- C29: renamed from C28; footprint (none) -> Capacitor_THT:C_Rect_L7.0mm_W2.5mm_P5.00mm
- C30: renamed from C32; footprint (none) -> Capacitor_THT:C_Rect_L7.0mm_W2.5mm_P5.00mm
- C31: renamed from C18; footprint (none) -> Capacitor_THT:C_Rect_L7.0mm_W2.5mm_P5.00mm
- C32: renamed from C23; footprint (none) -> Capacitor_THT:C_Rect_L7.0mm_W2.5mm_P5.00mm
- C33: renamed from C29; footprint (none) -> Capacitor_THT:C_Rect_L7.0mm_W2.5mm_P5.00mm
- C34: renamed from C33; footprint (none) -> Capacitor_THT:C_Rect_L7.0mm_W2.5mm_P5.00mm
- D12, D13, D14, D15: footprint (none) -> Diode_THT:D_DO-35_SOD27_P10.16mm_Horizontal
- L1, L2: footprint (none) -> Inductor_THT:L_Axial_L20.3mm_D12.7mm_P7.62mm_Vertical_Vishay_IHA-201
- R16: renamed from R19; footprint (none) -> Resistor_THT:R_Axial_DIN0207_L6.3mm_D2.5mm_P7.62mm_Horizontal
- R17: renamed from R26; footprint (none) -> Resistor_THT:R_Axial_DIN0207_L6.3mm_D2.5mm_P7.62mm_Horizontal
- R18: renamed from R16; footprint (none) -> Resistor_THT:R_Axial_DIN0207_L6.3mm_D2.5mm_P10.16mm_Horizontal
- R19: renamed from R20; footprint (none) -> Resistor_THT:R_Axial_DIN0207_L6.3mm_D2.5mm_P10.16mm_Horizontal
- R20: renamed from R23; footprint (none) -> Resistor_THT:R_Axial_DIN0207_L6.3mm_D2.5mm_P10.16mm_Horizontal
- R21: renamed from R27; footprint (none) -> Resistor_THT:R_Axial_DIN0207_L6.3mm_D2.5mm_P10.16mm_Horizontal
- R22: renamed from R21; footprint (none) -> Resistor_THT:R_Axial_DIN0207_L6.3mm_D2.5mm_P10.16mm_Horizontal
- R23: renamed from R28; footprint (none) -> Resistor_THT:R_Axial_DIN0207_L6.3mm_D2.5mm_P10.16mm_Horizontal
- R24: renamed from R18; footprint (none) -> Resistor_THT:R_Axial_DIN0207_L6.3mm_D2.5mm_P10.16mm_Horizontal
- R25: footprint (none) -> Resistor_THT:R_Axial_DIN0207_L6.3mm_D2.5mm_P10.16mm_Horizontal
- R26: renamed from R22; footprint (none) -> Resistor_THT:R_Axial_DIN0207_L6.3mm_D2.5mm_P10.16mm_Horizontal
- R27: renamed from R29; footprint (none) -> Resistor_THT:R_Axial_DIN0207_L6.3mm_D2.5mm_P10.16mm_Horizontal
- U4: renamed from U6; symbol calidus-rescue:TDA7293-tda7293 -> tda7293:TDA7293
- U5: renamed from U7; symbol calidus-rescue:TDA7293-tda7293 -> tda7293:TDA7293
- gave numbers to parts that had none: 5
- renumbered C27 to C14, C25 to C19, C37 to C20, C20 to C25, C19 to C35, C24 to C36, C30 to C37, C34 to C38, R14 to R28
Connections:
- net GNDS: no longer C14.2, R18.1, U4.4 (SIG_GND)
- new net: C?.1, R18.1, R?.1, U4.3 (+)
- new net: C13.1, R?.2
- new net ingnd_l: C14.2, C?.2, R18.2, U4.4 (SIG_GND)
Other:
- moved on the sheet: R18
