File: calidus_amp/calidus/psupply.sch (KiCad schematic (older format))
At the start: 42 parts, among them U1 LM317_3PinPackage, U2 LM337_TO220, U3 L7805

Commit message: WIP: Component placement
Parts:
- D1, D10, D11, D2, D3, D4, D7, D9: footprint Diode_THT:D_DO-41_SOD81_P7.62mm_Horizontal -> Diode_THT:D_DO-41_SOD81_P10.16mm_Horizontal
Changed lines of the file:
@@
 F 0 "D1" H 7050 1116 50  0000 C CNN
 F 1 "BZX85C20" H 7050 1025 50  0000 C CNN
-F 2 "Diode_THT:D_DO-41_SOD81_P7.62mm_Horizontal" H 7050 900 50  0001 C CNN
+F 2 "Diode_THT:D_DO-41_SOD81_P10.16mm_Horizontal" H 7050 900 50  0001 C CNN
 F 3 "~" H 7050 900 50  0001 C CNN
 	1    7050 900
@@
 F 0 "D11" H 7050 4484 50  0000 C CNN
 F 1 "BZX85C20" H 7050 4575 50  0000 C CNN
-F 2 "Diode_THT:D_DO-41_SOD81_P7.62mm_Horizontal" H 7050 4700 50  0001 C CNN
+F 2 "Diode_THT:D_DO-41_SOD81_P10.16mm_Horizontal" H 7050 4700 50  0001 C CNN
 F 3 "~" H 7050 4700 50  0001 C CNN
 	1    7050 4700
@@
 F 0 "D4" V 4854 1829 50  0000 L CNN
 F 1 "1N4007" V 4945 1829 50  0000 L CNN
-F 2 "Diode_THT:D_DO-41_SOD81_P7.62mm_Horizontal" H 4900 1750 50  0001 C CNN
+F 2 "Diode_THT:D_DO-41_SOD81_P10.16mm_Horizontal" H 4900 1750 50  0001 C CNN
 F 3 "~" H 4900 1750 50  0001 C CNN
 	1    4900 1750
@@
 F 0 "D3" H 5200 1284 50  0000 C CNN
 F 1 "1N4007" H 5200 1375 50  0000 C CNN
-F 2 "Diode_THT:D_DO-41_SOD81_P7.62mm_Horizontal" H 5200 1500 50  0001 C CNN
+F 2 "Diode_THT:D_DO-41_SOD81_P10.16mm_Horizontal" H 5200 1500 50  0001 C CNN
 F 3 "~" H 5200 1500 50  0001 C CNN
 	1    5200 1500
@@
 F 0 "D7" V 4854 3929 50  0000 L CNN
 F 1 "1N4007" V 4945 3929 50  0000 L CNN
-F 2 "Diode_THT:D_DO-41_SOD81_P7.62mm_Horizontal" H 4900 3850 50  0001 C CNN
+F 2 "Diode_THT:D_DO-41_SOD81_P10.16mm_Horizontal" H 4900 3850 50  0001 C CNN
 F 3 "~" H 4900 3850 50  0001 C CNN
 	1    4900 3850
@@
 F 0 "D9" H 5200 3976 50  0000 C CNN
 F 1 "1N4007" H 5200 3885 50  0000 C CNN
-F 2 "Diode_THT:D_DO-41_SOD81_P7.62mm_Horizontal" H 5200 4100 50  0001 C CNN
+F 2 "Diode_THT:D_DO-41_SOD81_P10.16mm_Horizontal" H 5200 4100 50  0001 C CNN
 F 3 "~" H 5200 4100 50  0001 C CNN
 	1    5200 4100
@@
 F 0 "D2" H 6350 1416 50  0000 C CNN
 F 1 "1N4007" H 6350 1325 50  0000 C CNN
-F 2 "Diode_THT:D_DO-41_SOD81_P7.62mm_Horizontal" H 6350 1200 50  0001 C CNN
+F 2 "Diode_THT:D_DO-41_SOD81_P10.16mm_Horizontal" H 6350 1200 50  0001 C CNN
 F 3 "~" H 6350 1200 50  0001 C CNN
 	1    6350 1200
@@
 F 0 "D10" H 6350 4524 50  0000 C CNN
 F 1 "1N4007" H 6350 4615 50  0000 C CNN
-F 2 "Diode_THT:D_DO-41_SOD81_P7.62mm_Horizontal" H 6350 4400 50  0001 C CNN
+F 2 "Diode_THT:D_DO-41_SOD81_P10.16mm_Horizontal" H 6350 4400 50  0001 C CNN
 F 3 "~" H 6350 4400 50  0001 C CNN
 	1    6350 4400

Commit message: WIP: Component placement and footpring assignment
Parts:
- C2, C9: Supplier Farnell:2943922 -> (none); Supplier1 (none) -> Farnell:2943922
- C3, C6: Manufacturer (none) -> Epcos:B41252B7109M000; Supplier1 (none) -> Farnell:2750101
- C5, C8: footprint Capacitor_THT:CP_Radial_D10.0mm_P5.00mm -> Capacitor_THT:CP_Radial_D6.3mm_P2.50mm; Manufacturer Rybicon:100YXF47MEFC10X16 -> Rybicon:50YXF47MEFC6.3X11; Supplier1 Farnell:1144641 -> Farnell:1144633; Voltage 100V -> 50V
Changed lines of the file:
@@
 F 1 "10m" H 4418 2550 50  0000 L CNN
 F 2 "Capacitor_THT:CP_Radial_D30.0mm_P10.00mm_SnapIn" H 4338 2400 50  0001 C CNN
-F 3 "~" H 4300 2550 50  0001 C CNN
+F 3 "http://www.farnell.com/datasheets/2280821.pdf" H 4300 2550 50  0001 C CNN
 F 4 "35V" H 4418 2459 50  0000 L CNN "Voltage"
+F 5 "Epcos:B41252B7109M000" H 4300 2550 50  0001 C CNN "Manufacturer"
+F 6 "Farnell:2750101" H 4300 2550 50  0001 C CNN "Supplier1"
 	1    4300 2550
 	1    0    0    -1
@@
 	-1   0    0    1
 $EndComp
-$Comp
-L Device:CP C5
-U 1 1 5C3CB3E8
-P 7600 2550
-F 0 "C5" H 7482 2641 50  0000 R CNN
-F 1 "47u" H 7482 2550 50  0000 R CNN
-F 2 "Capacitor_THT:CP_Radial_D10.0mm_P5.00mm" H 7638 2400 50  0001 C CNN
-F 3 "http://www.farnell.com/datasheets/2124421.pdf" H 7600 2550 50  0001 C CNN
-F 4 "100V" H 7482 2459 50  0000 R CNN "Voltage"
-F 5 "Rybicon:100YXF47MEFC10X16" H 7600 2550 50  0001 C CNN "Manufacturer"
-F 6 "Farnell:1144641" H 7600 2550 50  0001 C CNN "Supplier1"
-	1    7600 2550
-	-1   0    0    -1
-$EndComp
 Wire Wire Line
 	4150 1500 4450 1500
@@
 $EndComp
 $Comp
-L Device:CP C6
-U 1 1 5C45A6BB
-P 4300 3050
-F 0 "C6" H 4418 3141 50  0000 L CNN
-F 1 "10m" H 4418 3050 50  0000 L CNN
-F 2 "Capacitor_THT:CP_Radial_D30.0mm_P10.00mm_SnapIn" H 4338 2900 50  0001 C CNN
-F 3 "~" H 4300 3050 50  0001 C CNN
-F 4 "35V" H 4418 2959 50  0000 L CNN "Voltage"
-	1    4300 3050
-	1    0    0    -1
-$EndComp
-$Comp
 L power:GNDPWR #PWR08
 U 1 1 5C45ABCE
@@
 F 5 "X1" H 2415 2014 50  0000 L CNN "Type"
 F 6 "Kemet:PHE844RD6220MR06L2" H 2300 2150 50  0001 C CNN "Manufacturer"
-F 7 "Farnell:2943922" H 2300 2150 50  0001 C CNN "Supplier"
+F 7 "Farnell:2943922" H 2300 2150 50  0001 C CNN "Supplier1"
 	1    2300 2150
 	1    0    0    -1
@@
 F 5 "X1" H 2415 3314 50  0000 L CNN "Type"
 F 6 "Kemet:PHE844RD6220MR06L2" H 2300 3450 50  0001 C CNN "Manufacturer"
-F 7 "Farnell:2943922" H 2300 3450 50  0001 C CNN "Supplier"
+F 7 "Farnell:2943922" H 2300 3450 50  0001 C CNN "Supplier1"
 	1    2300 3450
 	1    0    0    -1
@@
 $EndComp
 $Comp
-L Device:CP C8
-U 1 1 5C5B32B4
-P 7600 3050
-F 0 "C8" H 7482 3141 50  0000 R CNN
-F 1 "47u" H 7482 3050 50  0000 R CNN
-F 2 "Capacitor_THT:CP_Radial_D10.0mm_P5.00mm" H 7638 2900 50  0001 C CNN
-F 3 "http://www.farnell.com/datasheets/2124421.pdf" H 7600 3050 50  0001 C CNN
-F 4 "100V" H 7482 2959 50  0000 R CNN "Voltage"
-F 5 "Rybicon:100YXF47MEFC10X16" H 7600 3050 50  0001 C CNN "Manufacturer"
-F 6 "Farnell:1144641" H 7600 3050 50  0001 C CNN "Supplier1"
-	1    7600 3050
-	-1   0    0    -1
-$EndComp
-$Comp
 L Device:CP C4
 U 1 1 5C5DD036
@@
 Wire Wire Line
 	2100 7100 2250 7100
+$Comp
+L Device:CP C6
+U 1 1 5C51F768
+P 4300 3050
+F 0 "C6" H 4418 3141 50  0000 L CNN
+F 1 "10m" H 4418 3050 50  0000 L CNN
+F 2 "Capacitor_THT:CP_Radial_D30.0mm_P10.00mm_SnapIn" H 4338 2900 50  0001 C CNN
+F 3 "http://www.farnell.com/datasheets/2280821.pdf" H 4300 3050 50  0001 C CNN
+F 4 "35V" H 4418 2959 50  0000 L CNN "Voltage"
+F 5 "Epcos:B41252B7109M000" H 4300 3050 50  0001 C CNN "Manufacturer"
+F 6 "Farnell:2750101" H 4300 3050 50  0001 C CNN "Supplier1"
+	1    4300 3050
+	1    0    0    -1
+$EndComp
+$Comp
+L Device:CP C5
+U 1 1 5C52E228
+P 7600 2550
+AR Path="/5C37BC48/5C52E228" Ref="C5"  Part="1"
+AR Path="/5C37BC7C/5C52E228" Ref="C?"  Part="1"
+F 0 "C5" H 7482 2641 50  0000 R CNN
+F 1 "47u" H 7482 2550 50  0000 R CNN
+F 2 "Capacitor_THT:CP_Radial_D6.3mm_P2.50mm" H 7638 2400 50  0001 C CNN
+F 3 "http://www.farnell.com/datasheets/2321304.pdf" H 7600 2550 50  0001 C CNN
+F 4 "50V" H 7482 2459 50  0000 R CNN "Voltage"
+F 5 "Rybicon:50YXF47MEFC6.3X11" H 7600 2550 50  0001 C CNN "Manufacturer"
+F 6 "Farnell:1144633" H 7600 2550 50  0001 C CNN "Supplier1"
+	1    7600 2550
+	-1   0    0    -1
+$EndComp
+$Comp
+L Device:CP C8
+U 1 1 5C53391A
+P 7600 3050
+AR Path="/5C37BC48/5C53391A" Ref="C8"  Part="1"
+AR Path="/5C37BC7C/5C53391A" Ref="C?"  Part="1"
+F 0 "C8" H 7482 3141 50  0000 R CNN
+F 1 "47u" H 7482 3050 50  0000 R CNN
+F 2 "Capacitor_THT:CP_Radial_D6.3mm_P2.50mm" H 7638 2900 50  0001 C CNN
+F 3 "http://www.farnell.com/datasheets/2321304.pdf" H 7600 3050 50  0001 C CNN
+F 4 "50V" H 7482 2959 50  0000 R CNN "Voltage"
+F 5 "Rybicon:50YXF47MEFC6.3X11" H 7600 3050 50  0001 C CNN "Manufacturer"
+F 6 "Farnell:1144633" H 7600 3050 50  0001 C CNN "Supplier1"
+	1    7600 3050
+	-1   0    0    -1
+$EndComp
 $EndSCHEMATC

Commit message: WIP: Component placement and footprint assignement
- Finished all capacitors
- Finished all ICs
Parts:
- C10, C7: Supplier Farnell:1144639 -> (none); Supplier1 (none) -> Farnell:1144639
- R15, R16: Manufacturer (none) -> TE Connectivity:LR1F10R; Power 1/4 -> 0.6W; Supplier1 (none) -> Farnell:2329993
- U1: value LM317_3PinPackage -> LM317; Manufacturer (none) -> ON Semiconductor:LM317BTG; Supplier1 (none) -> Farnell:1214459
- U2: value LM337_TO220 -> LM337; Manufacturer (none) -> ON Semiconductor:LM337BTG; Supplier1 (none) -> Farnell:1652327
- U3: Manufacturer (none) -> ST:L7805ACV; Supplier1 (none) -> Farnell:1087086
Changed lines of the file:
@@
 P 6700 1500
 F 0 "U1" H 6700 1742 50  0000 C CNN
-F 1 "LM317_3PinPackage" H 6700 1651 50  0000 C CNN
+F 1 "LM317" H 6700 1651 50  0000 C CNN
 F 2 "Package_TO_SOT_THT:TO-220-3_Vertical" H 6700 1750 50  0001 C CIN
 F 3 "http://www.ti.com/lit/ds/symlink/lm317.pdf" H 6700 1500 50  0001 C CNN
+F 4 "ON Semiconductor:LM317BTG " H 0   0   50  0001 C CNN "Manufacturer"
+F 5 "Farnell:1214459" H 0   0   50  0001 C CNN "Supplier1"
 	1    6700 1500
 	1    0    0    -1
@@
 	2700 6300 2800 6300
 Connection ~ 2000 2800
-$Comp
-L Device:R R15
-U 1 1 5C46F465
-P 2400 6300
-F 0 "R15" V 2011 6300 50  0000 C CNN
-F 1 "10" V 2102 6300 50  0000 C CNN
-F 2 "Resistor_THT:R_Axial_DIN0207_L6.3mm_D2.5mm_P10.16mm_Horizontal" V 2330 6300 50  0001 C CNN
-F 3 "~" H 2400 6300 50  0001 C CNN
-F 4 "1/4" V 2193 6300 50  0000 C CNN "Power"
-F 5 "MF" V 2284 6300 50  0000 C CNN "Type"
-	1    2400 6300
-	0    1    1    0
-$EndComp
 Wire Wire Line
 	2550 6300 2700 6300
@@
 P 6700 4100
 F 0 "U2" H 6700 3950 50  0000 C CNN
-F 1 "LM337_TO220" H 6700 3859 50  0000 C CNN
+F 1 "LM337" H 6700 3859 50  0000 C CNN
 F 2 "Package_TO_SOT_THT:TO-220-3_Vertical" H 6700 3900 50  0001 C CIN
 F 3 "http://www.ti.com/lit/ds/symlink/lm337-n.pdf" H 6700 4100 50  0001 C CNN
+F 4 "ON Semiconductor:LM337BTG" H 0   0   50  0001 C CNN "Manufacturer"
+F 5 "Farnell:1652327" H 0   0   50  0001 C CNN "Supplier1"
 	1    6700 4100
 	1    0    0    -1
@@
 F 2 "Package_TO_SOT_THT:TO-220-3_Vertical" H 5525 5950 50  0001 L CIN
 F 3 "http://www.st.com/content/ccc/resource/technical/document/datasheet/41/4f/b3/b0/12/d4/47/88/CD00000444.pdf/files/CD00000444.pdf/jcr:content/translations/en.CD00000444.pdf" H 5500 6050 50  0001 C CNN
+F 4 "ST:L7805ACV" H 0   0   50  0001 C CNN "Manufacturer"
+F 5 "Farnell:1087086" H 0   0   50  0001 C CNN "Supplier1"
 	1    5500 6100
 	1    0    0    -1
@@
 F 4 "63V" H 5382 2959 50  0000 R CNN "Voltage"
 F 5 "Rybicon:63YXF470MEFC12.5X25" V 5500 3050 50  0001 C CNN "Manufacturer"
-F 6 "Farnell:1144639" V 5500 3050 50  0001 C CNN "Supplier"
+F 6 "" V 5500 3050 50  0001 C CNN "Supplier"
+F 7 "Farnell:1144639" H 0   0   50  0001 C CNN "Supplier1"
 	1    5500 3050
 	-1   0    0    -1
@@
 F 4 "63V" V 4450 4100 50  0000 C CNN "Voltage"
 F 5 "Rybicon:63YXF470MEFC12.5X25" V 4600 4100 50  0001 C CNN "Manufacturer"
-F 6 "Farnell:1144639" V 4600 4100 50  0001 C CNN "Supplier"
+F 6 "" V 4600 4100 50  0001 C CNN "Supplier"
+F 7 "Farnell:1144639" H 0   0   50  0001 C CNN "Supplier1"
 	1    4600 4100
 	0    -1   1    0
@@
 Wire Wire Line
 	2700 7100 2800 7100
-$Comp
-L Device:R R16
-U 1 1 5C4F636E
-P 2400 7100
-F 0 "R16" V 2011 7100 50  0000 C CNN
-F 1 "10" V 2102 7100 50  0000 C CNN
-F 2 "Resistor_THT:R_Axial_DIN0207_L6.3mm_D2.5mm_P10.16mm_Horizontal" V 2330 7100 50  0001 C CNN
-F 3 "~" H 2400 7100 50  0001 C CNN
-F 4 "1/4" V 2193 7100 50  0000 C CNN "Power"
-F 5 "MF" V 2284 7100 50  0000 C CNN "Type"
-	1    2400 7100
-	0    1    1    0
-$EndComp
 Wire Wire Line
 	2550 7100 2700 7100
@@
 	-1   0    0    -1
 $EndComp
+$Comp
+L Device:R R?
+U 1 1 5C532B5E
+P 2400 6300
+AR Path="/5C37BC7C/5C532B5E" Ref="R?"  Part="1"
+AR Path="/5C37BC48/5C532B5E" Ref="R15"  Part="1"
+F 0 "R15" V 2011 6300 50  0000 C CNN
+F 1 "10" V 2102 6300 50  0000 C CNN
+F 2 "Resistor_THT:R_Axial_DIN0207_L6.3mm_D2.5mm_P10.16mm_Horizontal" V 2330 6300 50  0001 C CNN
+F 3 "http://www.farnell.com/datasheets/1723855.pdf" H 2400 6300 50  0001 C CNN
+F 4 "0.6W" V 2193 6300 50  0000 C CNN "Power"
+F 5 "MF" V 2284 6300 50  0000 C CNN "Type"
+F 6 "TE Connectivity:LR1F10R" H 2400 6300 50  0001 C CNN "Manufacturer"
+F 7 "Farnell:2329993" H 2400 6300 50  0001 C CNN "Supplier1"
+	1    2400 6300
+	0    1    1    0
+$EndComp
+$Comp
+L Device:R R?
+U 1 1 5C53820F
+P 2400 7100
+AR Path="/5C37BC7C/5C53820F" Ref="R?"  Part="1"
+AR Path="/5C37BC48/5C53820F" Ref="R16"  Part="1"
+F 0 "R16" V 2011 7100 50  0000 C CNN
+F 1 "10" V 2102 7100 50  0000 C CNN
+F 2 "Resistor_THT:R_Axial_DIN0207_L6.3mm_D2.5mm_P10.16mm_Horizontal" V 2330 7100 50  0001 C CNN
+F 3 "http://www.farnell.com/datasheets/1723855.pdf" H 2400 7100 50  0001 C CNN
+F 4 "0.6W" V 2193 7100 50  0000 C CNN "Power"
+F 5 "MF" V 2284 7100 50  0000 C CNN "Type"
+F 6 "TE Connectivity:LR1F10R" H 2400 7100 50  0001 C CNN "Manufacturer"
+F 7 "Farnell:2329993" H 2400 7100 50  0001 C CNN "Supplier1"
+	1    2400 7100
+	0    1    1    0
+$EndComp
 $EndSCHEMATC
