File: calidus_amp/calidus/calidus.kicad_pcb (KiCad board)
At the start: 4 copper layers, 140 x 110 mm, 134 parts, among them J1 left_out, J10 led_power, J11 sense_bus, J2 power, J3 input, J4 right_out, J5 prevs, J6 icsp, J7 mute_key, J8 led_overload, J9 service, Q1 Q_NPN_CBE, Q2 Q_NPN_CBE, Q3 Q_NPN_CBE, U1 LM317, U2 LM337, U3 L7805, U4 TDA7293, U5 TDA7293, U6 PIC18F26K42-I/SP

Commit message: WIP: Minor placement adjustements
Parts:
- moved D12 10.8 mm to (118.6, 52.2), turned to 90 degrees
- moved C22 5.08 mm to (155.7, 63.0), turned to 0 degrees
- moved D13 3.31 mm to (121.1, 44.6)
- moved C35 2.50 mm to (150.6, 57.3), turned to 180 degrees
- moved D14 0.90 mm to (178.6, 52.2)
- moved D15 0.90 mm to (181.1, 44.6)
- moved L1 0.31 mm to (110.3, 46.5)
- moved J3 0.13 mm to (56.0, 72.6)
- moved J5 0.13 mm to (56.0, 87.2)
- moved J2 0.13 mm to (184.0, 115.1)
- moved C16 0.08 mm to (160.7, 52.2)
Changed lines of the file:
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@@
   )
   (module Diode_THT:D_DO-35_SOD27_P7.62mm_Horizontal (layer F.Cu)
-    (at 181.75 43.97 270)
+    (at 181.115 44.605 270)
     (descr "Diode, DO-35_SOD27 series, Axial, Horizontal, pin pitch=7.62mm, , length*diameter=4*2mm^2, , http://www.diodes.com/_files/packages/DO-35.pdf")
     (tags "Diode DO-35_SOD27 series Axial Horizontal pin pitch 7.62mm  length 4mm diameter 2mm")
@@
   )
   (module Diode_THT:D_DO-35_SOD27_P7.62mm_Horizontal (layer F.Cu)
-    (at 179.21 51.59 90)
+    (at 178.575 52.225 90)
     (descr "Diode, DO-35_SOD27 series, Axial, Horizontal, pin pitch=7.62mm, , length*diameter=4*2mm^2, , http://www.diodes.com/_files/packages/DO-35.pdf")
     (tags "Diode DO-35_SOD27 series Axial Horizontal pin pitch 7.62mm  length 4mm diameter 2mm")
@@
   )
   (module Inductor_THT:L_Axial_L20.3mm_D12.7mm_P7.62mm_Vertical_Vishay_IHA-201 (layer F.Cu)
-    (at 110.63 46.51 180)
+    (at 110.32 46.51 180)
     (descr "Inductor, Axial series, Axial, Vertical, pin pitch=7.62mm, , length*diameter=20.32*12.7mm^2, Vishay, IHA-201, http://www.vishay.com/docs/34014/iha.pdf")
     (tags "Inductor Axial series Axial Vertical pin pitch 7.62mm  length 20.32mm diameter 12.7mm Vishay IHA-201")
@@
   )
   (module Connector_Phoenix_MC:PhoenixContact_MCV_1,5_3-G-3.5_1x03_P3.50mm_Vertical locked (layer F.Cu)
-    (at 55.865 87.165 90)
+    (at 56 87.165 90)
     (descr "Generic Phoenix Contact connector footprint for: MCV_1,5/3-G-3.5; number of pins: 03; pin pitch: 3.50mm; Vertical || order number: 1843619 8A 160V")
     (tags "phoenix_contact connector MCV_01x03_G_3.5mm")
@@
   )
   (module Capacitor_THT:CP_Radial_D10.0mm_P5.00mm (layer F.Cu)
-    (at 160.795 52.225 180)
+    (at 160.715 52.225 180)
     (descr "CP, Radial series, Radial, pin pitch=5.00mm, , diameter=10mm, Electrolytic Capacitor")
     (tags "CP Radial series Radial pin pitch 5.00mm  diameter 10mm Electrolytic Capacitor")
@@
   )
   (module Capacitor_THT:CP_Radial_D10.0mm_P5.00mm (layer F.Cu)
-    (at 160.795 63.02 180)
+    (at 155.715 63.02)
     (descr "CP, Radial series, Radial, pin pitch=5.00mm, , diameter=10mm, Electrolytic Capacitor")
     (tags "CP Radial series Radial pin pitch 5.00mm  diameter 10mm Electrolytic Capacitor")
-    (fp_text reference C22 (at 2.5 -6.25 180) (layer F.SilkS)
+    (fp_text reference C22 (at 2.5 -6.25) (layer F.SilkS)
       (effects (font (size 1 1) (thickness 0.15)))
     )
-    (fp_text value 220u (at 2.5 6.25 180) (layer F.Fab)
+    (fp_text value 220u (at 2.5 6.25) (layer F.Fab)
       (effects (font (size 1 1) (thickness 0.15)))
     )
@@
     (fp_line (start -2.979646 -2.875) (end -1.979646 -2.875) (layer F.SilkS) (width 0.12))
     (fp_line (start -2.479646 -3.375) (end -2.479646 -2.375) (layer F.SilkS) (width 0.12))
-    (fp_text user %R (at 2.5 0 180) (layer F.Fab)
+    (fp_text user %R (at 2.5 0) (layer F.Fab)
       (effects (font (size 1 1) (thickness 0.15)))
     )
-    (pad 1 thru_hole rect (at 0 0 180) (size 2 2) (drill 1) (layers *.Cu *.Mask)
+    (pad 1 thru_hole rect (at 0 0) (size 2 2) (drill 1) (layers *.Cu *.Mask)
       (net 2 Earth_Protective))
-    (pad 2 thru_hole circle (at 5 0 180) (size 2 2) (drill 1) (layers *.Cu *.Mask)
+    (pad 2 thru_hole circle (at 5 0) (size 2 2) (drill 1) (layers *.Cu *.Mask)
       (net 3 -pwvs))
     (model ${KISYS3DMOD}/Capacitor_THT.3dshapes/CP_Radial_D10.0mm_P5.00mm.wrl
@@
   )
   (module Diode_THT:D_DO-35_SOD27_P7.62mm_Horizontal (layer F.Cu)
-    (at 119.52 41.43 270)
+    (at 118.575 52.225 90)
     (descr "Diode, DO-35_SOD27 series, Axial, Horizontal, pin pitch=7.62mm, , length*diameter=4*2mm^2, , http://www.diodes.com/_files/packages/DO-35.pdf")
     (tags "Diode DO-35_SOD27 series Axial Horizontal pin pitch 7.62mm  length 4mm diameter 2mm")
-    (fp_text reference D12 (at 3.81 -2.12 270) (layer F.SilkS)
+    (fp_text reference D12 (at 3.81 -2.12 90) (layer F.SilkS)
       (effects (font (size 1 1) (thickness 0.15)))
     )
-    (fp_text value 1N5404 (at 3.81 2.12 270) (layer F.Fab)
+    (fp_text value 1N5404 (at 3.81 2.12 90) (layer F.Fab)
       (effects (font (size 1 1) (thickness 0.15)))
     )
@@
     (fp_line (start 8.67 1.25) (end 8.67 -1.25) (layer F.CrtYd) (width 0.05))
     (fp_line (start 8.67 -1.25) (end -1.05 -1.25) (layer F.CrtYd) (width 0.05))
-    (fp_text user %R (at 4.11 0 270) (layer F.Fab)
+    (fp_text user %R (at 4.11 0 90) (layer F.Fab)
       (effects (font (size 0.8 0.8) (thickness 0.12)))
     )
-    (fp_text user K (at 0 -1.8 270) (layer F.Fab)
+    (fp_text user K (at 0 -1.8 90) (layer F.Fab)
       (effects (font (size 1 1) (thickness 0.15)))
     )
-    (fp_text user K (at 0 -1.8 270) (layer F.SilkS)
+    (fp_text user K (at 0 -1.8 90) (layer F.SilkS)
       (effects (font (size 1 1) (thickness 0.15)))
     )
-    (pad 1 thru_hole rect (at 0 0 270) (size 1.6 1.6) (drill 0.8) (layers *.Cu *.Mask)
+    (pad 1 thru_hole rect (at 0 0 90) (size 1.6 1.6) (drill 0.8) (layers *.Cu *.Mask)
       (net 1 +pwvs))
-    (pad 2 thru_hole oval (at 7.62 0 270) (size 1.6 1.6) (drill 0.8) (layers *.Cu *.Mask)
+    (pad 2 thru_hole oval (at 7.62 0 90) (size 1.6 1.6) (drill 0.8) (layers *.Cu *.Mask)
       (net 65 "Net-(C31-Pad1)"))
     (model ${KISYS3DMOD}/Diode_THT.3dshapes/D_DO-35_SOD27_P7.62mm_Horizontal.wrl
@@
   )
   (module Diode_THT:D_DO-35_SOD27_P7.62mm_Horizontal (layer F.Cu)
-    (at 122.06 41.43 270)
+    (at 121.115 44.605 270)
     (descr "Diode, DO-35_SOD27 series, Axial, Horizontal, pin pitch=7.62mm, , length*diameter=4*2mm^2, , http://www.diodes.com/_files/packages/DO-35.pdf")
     (tags "Diode DO-35_SOD27 series Axial Horizontal pin pitch 7.62mm  length 4mm diameter 2mm")
@@
   )
   (module Connector_Phoenix_MC:PhoenixContact_MCV_1,5_3-G-3.81_1x03_P3.81mm_Vertical locked (layer F.Cu)
-    (at 184.135 115.09 270)
+    (at 184 115.09 270)
     (descr "Generic Phoenix Contact connector footprint for: MCV_1,5/3-G-3.81; number of pins: 03; pin pitch: 3.81mm; Vertical || order number: 1803439 8A 160V")
     (tags "phoenix_contact connector MCV_01x03_G_3.81mm")
@@
   )
   (module Connector_Phoenix_MC:PhoenixContact_MCV_1,5_4-G-3.5_1x04_P3.50mm_Vertical locked (layer F.Cu)
-    (at 55.865 72.56 90)
+    (at 56 72.56 90)
     (descr "Generic Phoenix Contact connector footprint for: MCV_1,5/4-G-3.5; number of pins: 04; pin pitch: 3.50mm; Vertical || order number: 1843622 8A 160V")
     (tags "phoenix_contact connector MCV_01x04_G_3.5mm")
@@
   )
   (module Capacitor_THT:CP_Radial_D6.3mm_P2.50mm (layer F.Cu)
-    (at 148.095 57.305)
+    (at 150.595 57.305 180)
     (descr "CP, Radial series, Radial, pin pitch=2.50mm, , diameter=6.3mm, Electrolytic Capacitor")
     (tags "CP Radial series Radial pin pitch 2.50mm  diameter 6.3mm Electrolytic Capacitor")
-    (fp_text reference C35 (at 1.25 -4.4) (layer F.SilkS)
+    (fp_text reference C35 (at 1.25 -4.4 180) (layer F.SilkS)
       (effects (font (size 1 1) (thickness 0.15)))
     )
-    (fp_text value 47u (at 1.25 4.4) (layer F.Fab)
+    (fp_text value 47u (at 1.25 4.4 180) (layer F.Fab)
       (effects (font (size 1 1) (thickness 0.15)))
     )
@@
     (fp_line (start -2.250241 -1.839) (end -1.620241 -1.839) (layer F.SilkS) (width 0.12))
     (fp_line (start -1.935241 -2.154) (end -1.935241 -1.524) (layer F.SilkS) (width 0.12))
-    (fp_text user %R (at 1.25 0) (layer F.Fab)
+    (fp_text user %R (at 1.25 0 180) (layer F.Fab)
       (effects (font (size 1 1) (thickness 0.15)))
     )
-    (pad 1 thru_hole rect (at 0 0) (size 1.6 1.6) (drill 0.8) (layers *.Cu *.Mask)
+    (pad 1 thru_hole rect (at 0 0 180) (size 1.6 1.6) (drill 0.8) (layers *.Cu *.Mask)
       (net 2 Earth_Protective))
-    (pad 2 thru_hole circle (at 2.5 0) (size 1.6 1.6) (drill 0.8) (layers *.Cu *.Mask)
+    (pad 2 thru_hole circle (at 2.5 0 180) (size 1.6 1.6) (drill 0.8) (layers *.Cu *.Mask)
       (net 8 -vs))
     (model ${KISYS3DMOD}/Capacitor_THT.3dshapes/CP_Radial_D6.3mm_P2.50mm.wrl

Commit message: WIP: Component placement.
Signed-off-by: Nenad Radulovic <nenad.b.radulovic@gmail.com>
Parts:
- moved D16 5.08 mm to (53.3, 110.0)
- moved C45 1.91 mm to (85.7, 111.9)
- moved R38 1.80 mm to (66.7, 118.9)
- moved R39 1.80 mm to (89.5, 96.0)
- moved R43 1.80 mm to (89.5, 124.0)
- moved R44 1.80 mm to (66.7, 124.0)
- moved C46 1.80 mm to (85.7, 116.4)
- moved R17 1.80 mm to (84.4, 101.1)
- moved R36 1.80 mm to (66.7, 91.0)
- moved R37 1.80 mm to (89.5, 108.7)
- moved R40 1.80 mm to (89.5, 93.5)
- moved R41 1.80 mm to (89.5, 91.0)
- moved R45 1.80 mm to (71.7, 121.4)
- moved R18 1.80 mm to (84.4, 98.6)
- moved R42 1.80 mm to (66.7, 116.4)
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Routing:
- net /Control and Monitoring Unit/ac_in: track 0.00 -> 19.9 mm
- net /psupply/pri_hi: track 0.00 -> 11.2 mm
